Commit message: Redid the URDF joints in Soldiworks to reflect some model changes. Reduced weight of vehicle and trailer to improve drive characteristics.

File: urdf/project_1_group_2.urdf.xacro (robot description, xacro)
@@ -39,15 +39,15 @@
     <inertial>
       <origin
-        xyz="0.219542185844718 -0.489097435985613 0.253171163731009"
-        rpy="0 0 0" />
-      <mass
-        value="10.0" />
-      <inertia
-        ixx="3.47370213259269"
-        ixy="8.68638754776676E-06"
-        ixz="1.2881777172653E-06"
-        iyy="1.51493007257673"
-        iyz="0.0559660105211113"
-        izz="4.32787408102169" />
+        xyz="0.219542184923656 0.253147662670064 0.488981343790689"
+        rpy="0 0 0" />
+      <mass
+        value="1" />
+      <inertia
+        ixx="3.47686976214323"
+        ixy="1.28363813560472E-06"
+        ixz="-8.67881754875189E-06"
+        iyy="4.33091580677011"
+        iyz="-0.0565812633669083"
+        izz="1.5150564663539" />
     </inertial>
     <visual>
@@ -79,15 +79,15 @@
     <inertial>
       <origin
-        xyz="2.8607507807088E-08 0.0723663419355983 0.0025405194968964"
-        rpy="0 0 0" />
-      <mass
-        value="0.295424107267105" />
-      <inertia
-        ixx="0.000710809060839364"
-        ixy="1.53957020724956E-10"
-        ixz="3.53322320619659E-10"
+        xyz="2.86075080291326E-08 -0.0749063419355981 -0.00254051949689645"
+        rpy="0 0 0" />
+      <mass
+        value="5.295424107267105" />
+      <inertia
+        ixx="0.000710809060839366"
+        ixy="-1.53957020615015E-10"
+        ixz="-3.53322320543782E-10"
         iyy="0.000104054571155282"
-        iyz="3.85934455800398E-05"
-        izz="0.00069010101560226" />
+        iyz="3.85934455800395E-05"
+        izz="0.000690101015602262" />
     </inertial>
     <visual>
@@ -119,6 +119,6 @@
     type="revolute">
     <origin
-      xyz="0.070952 -0.7342 0.038134"
-      rpy="1.5708 0 -1.6485" />
+      xyz="0.070952 -0.7342 0.035594"
+      rpy="-1.5708 0 -1.5708" />
     <parent
       link="base_link" />
@@ -128,8 +128,8 @@
       xyz="0 1 0" />
     <limit
-      lower="-0.7"
-      upper="0.7"
-      effort="100"
-      velocity="100" />
+      lower="-3.14"
+      upper="3.14"
+      effort="10"
+      velocity="10" />
   </joint>
   <link
@@ -137,15 +137,15 @@
     <inertial>
       <origin
-        xyz="-0.00233208035893656 0.0353869418204771 0.00100647960707934"
+        xyz="0 0.0251005990323743 0"
         rpy="0 0 0" />
       <mass
         value="0.217134053712094" />
       <inertia
-        ixx="0.000126052696684197"
-        ixy="-6.05628557286825E-20"
-        ixz="-3.3881317890172E-21"
+        ixx="0.000126052696684198"
+        ixy="-3.30911918449584E-21"
+        ixz="6.7762635780344E-21"
         iyy="0.000159854355976214"
-        iyz="-1.27901975035399E-19"
-        izz="0.000126052696684197" />
+        iyz="-7.03947290074457E-21"
+        izz="0.000126052696684198" />
     </inertial>
     <visual>
@@ -177,6 +177,6 @@
     type="continuous">
     <origin
-      xyz="0 0.023495 0.030481"
-      rpy="1.5708 0 1.1634" />
+      xyz="0 -0.0234950000000001 -0.040767"
+      rpy="-1.5707963267949 0 -1.16226628629428" />
     <parent
       link="steering_wheel_1" />
@@ -190,5 +190,5 @@
     <inertial>
       <origin
-        xyz="-0.00233208035893662 0.0356826852487729 0.00099954289455717"
+        xyz="0 0.0380963424606702 -6.9367125220543E-06"
         rpy="0 0 0" />
       <mass
@@ -196,8 +196,8 @@
       <inertia
         ixx="0.00664149361787531"
-        ixy="-5.28548559086683E-18"
-        ixz="-4.33680868994202E-19"
+        ixy="3.02337822610582E-19"
+        ixz="2.16840434497101E-19"
         iyy="0.0114725337233255"
-        iyz="5.01717636383912E-07"
+        iyz="5.01717636400841E-07"
         izz="0.00664244711710664" />
     </inertial>
@@ -227,8 +227,8 @@
   </link>
   <joint
-    name="tire_joint_1"
+    name="tire_1_joint"
     type="fixed">
     <origin
-      xyz="0 0 0"
+      xyz="0 -0.0127000000000001 0"
       rpy="0 0 0" />
     <parent
@@ -243,15 +243,15 @@
     <inertial>
       <origin
-        xyz="2.86075080291326E-08 0.0723663419355979 0.0025405194968961"
-        rpy="0 0 0" />
-      <mass
-        value="0.295424107267104" />
-      <inertia
-        ixx="0.000710809060839366"
-        ixy="1.53957022022187E-10"
-        ixz="3.53322320463805E-10"
+        xyz="2.86075079181103E-08 0.074906341935598 0.00254051949689649"
+        rpy="0 0 0" />
+      <mass
+        value="5.295424107267105" />
+      <inertia
+        ixx="0.000710809060839365"
+        ixy="1.53957021878157E-10"
+        ixz="3.53322320610221E-10"
         iyy="0.000104054571155282"
-        iyz="3.85934455800392E-05"
-        izz="0.000690101015602263" />
+        iyz="3.85934455800397E-05"
+        izz="0.000690101015602261" />
     </inertial>
     <visual>
@@ -283,6 +283,6 @@
     type="revolute">
     <origin
-      xyz="0.36813 -0.7342 0.038134"
-      rpy="1.5708 0 1.4699" />
+      xyz="0.36813 -0.7342 0.035594"
+      rpy="1.5708 0 1.5708" />
     <parent
       link="base_link" />
@@ -292,8 +292,8 @@
       xyz="0 1 0" />
     <limit
-      lower="-0.7"
-      upper="0.7"
+      lower="-3.14"
+      upper="3.14"
       effort="100"
-      velocity="100" />
+      velocity="10" />
   </joint>
   <link
@@ -301,5 +301,5 @@
     <inertial>
       <origin
-        xyz="-3.33066907387547E-16 0.0352804142384009 0.00254000000000009"
+        xyz="0 0.0251005990323743 0"
         rpy="0 0 0" />
       <mass
@@ -307,8 +307,8 @@
       <inertia
         ixx="0.000126052696684198"
-        ixy="-1.42301535138722E-19"
-        ixz="3.17002825963484E-22"
+        ixy="-2.42959470068895E-21"
+        ixz="0"
         iyy="0.000159854355976214"
-        iyz="4.53198898728574E-20"
+        iyz="-1.47427383956479E-20"
         izz="0.000126052696684198" />
     </inertial>
@@ -341,6 +341,6 @@
     type="continuous">
     <origin
-      xyz="0 0.023495 0.030587184793973"
-      rpy="1.5707963267949 0 0" />
+      xyz="0 0.0234950000000022 0.0407670000000003"
+      rpy="1.5707963267949 0 0.927408187420047" />
     <parent
       link="steering_wheel_2" />
@@ -354,14 +354,14 @@
     <inertial>
       <origin
-        xyz="-1.11022302462516E-16 0.0355761576666964 0.002533063287478"
+        xyz="-5.55111512312578E-17 0.0380963424606702 -6.93671252216532E-06"
         rpy="0 0 0" />
       <mass
         value="1.9636352752673" />
       <inertia
-        ixx="0.00664149361787531"
-        ixy="-2.24429849704499E-17"
-        ixz="-1.96935160236779E-20"
+        ixx="0.00664149361787532"
+        ixy="5.1086674631275E-20"
+        ixz="-2.16840434497101E-19"
         iyy="0.0114725337233255"
-        iyz="5.01717636407577E-07"
+        iyz="5.01717636401181E-07"
         izz="0.00664244711710664" />
     </inertial>
@@ -394,5 +394,5 @@
     type="fixed">
     <origin
-      xyz="0 0 0"
+      xyz="0 -0.0126999999999999 0"
       rpy="0 0 0" />
     <parent
@@ -407,5 +407,5 @@
     <inertial>
       <origin
-        xyz="-3.46944695195361E-17 -0.00140110038134092 2.77555756156289E-17"
+        xyz="0 -0.00140110038134092 0"
         rpy="0 0 0" />
       <mass
@@ -413,8 +413,8 @@
       <inertia
         ixx="0.000126052696684197"
-        ixy="3.65602981705437E-21"
-        ixz="-1.01643953670516E-20"
+        ixy="3.65980047539585E-21"
+        ixz="-6.7762635780344E-21"
         iyy="0.000159854355976214"
-        iyz="-7.36513260038282E-22"
+        iyz="-7.39817207392887E-22"
         izz="0.000126052696684197" />
     </inertial>
@@ -455,8 +455,4 @@
     <axis
       xyz="0 1 0" />
-      <limit
-      effort="100"
-      velocity="1000"
-      />
   </joint>
   <link
@@ -464,5 +460,5 @@
     <inertial>
       <origin
-        xyz="2.08166817117217E-17 0.048894643046955 -6.93671252216532E-06"
+        xyz="2.08166817117217E-17 0.0380963424606702 -6.93671252210981E-06"
         rpy="0 0 0" />
       <mass
@@ -470,6 +466,6 @@
       <inertia
         ixx="0.00664149361787532"
-        ixy="6.09863722023096E-19"
-        ixz="6.50521303491303E-19"
+        ixy="6.09678433565884E-19"
+        ixz="8.67361737988404E-19"
         iyy="0.0114725337233256"
         iyz="5.01717636401377E-07"
@@ -501,8 +497,8 @@
   </link>
   <joint
-    name="drive_tire_joint"
+    name="drive_tire_1_joint"
     type="fixed">
     <origin
-      xyz="0 -0.05 0"
+      xyz="0 -0.0392016994137152 0"
       rpy="0 0 0" />
     <parent
@@ -517,14 +513,14 @@
     <inertial>
       <origin
-        xyz="-2.77555756156289E-17 0.0276405990323743 0"
+        xyz="0 0.0251005990323744 0"
         rpy="0 0 0" />
       <mass
         value="0.217134053712094" />
       <inertia
-        ixx="0.000126052696684198"
-        ixy="-3.68451216035455E-22"
-        ixz="3.3881317890172E-21"
+        ixx="0.000126052696684197"
+        ixy="-5.05000906564327E-21"
+        ixz="1.01643953670516E-20"
         iyy="0.000159854355976214"
-        iyz="4.59516996223815E-21"
+        iyz="3.01026101938204E-21"
         izz="0.000126052696684198" />
     </inertial>
@@ -557,6 +553,6 @@
     type="continuous">
     <origin
-      xyz="0.41004 -0.2262 0.061675"
-      rpy="0 0.13365 -1.5708" />
+      xyz="0.41258 -0.2262 0.061675"
+      rpy="0 0.9434 -1.5708" />
     <parent
       link="base_link" />
@@ -565,8 +561,4 @@
     <axis
       xyz="0 1 0" />
-      <limit
-      effort="100"
-      velocity="1000"
-      />
   </joint>
   <link
@@ -574,5 +566,5 @@
     <inertial>
       <origin
-        xyz="1.11022302462516E-16 0.0406363424606702 -6.93671252208206E-06"
+        xyz="2.77555756156289E-17 0.0380963424606702 -6.93671252208206E-06"
         rpy="0 0 0" />
       <mass
@@ -580,8 +572,8 @@
       <inertia
         ixx="0.00664149361787531"
-        ixy="-2.07046616044473E-19"
-        ixz="-1.62630325872826E-19"
+        ixy="3.34048618573415E-19"
+        ixz="6.50521303491303E-19"
         iyy="0.0114725337233255"
-        iyz="5.01717636401017E-07"
+        iyz="5.0171763640111E-07"
         izz="0.00664244711710664" />
     </inertial>
@@ -614,5 +606,5 @@
     type="fixed">
     <origin
-      xyz="0 -0.0127 0"
+      xyz="0 -0.0126999999999999 0"
       rpy="3.14159265358979 0 3.14159265358979" />
     <parent
@@ -627,15 +619,15 @@
     <inertial>
       <origin
-        xyz="1.03723919092635E-07 0.039678899062889 0.429404896824893"
-        rpy="0 0 0" />
-      <mass
-        value="5.43041573976378" />
-      <inertia
-        ixx="0.10730066092027"
-        ixy="3.55141031738537E-09"
-        ixz="1.34013193767086E-07"
-        iyy="0.205190385513249"
-        iyz="-0.00161014497039631"
-        izz="0.111162712366413" />
+        xyz="-2.14872014431267E-07 0.122240676993307 0.407195343988752"
+        rpy="0 0 0" />
+      <mass
+        value=".5" />
+      <inertia
+        ixx="0.106926412723749"
+        ixy="-2.14631197863797E-08"
+        ixz="-2.44065610516401E-07"
+        iyy="0.204818186461493"
+        iyz="-0.00158445646443877"
+        izz="0.111161118457744" />
     </inertial>
     <visual>
@@ -667,5 +659,5 @@
     type="continuous">
     <origin
-      xyz="0.21954 0.075693 0.11822"
+      xyz="0.21954 0.093844 0.041004"
       rpy="1.5708 0 3.1416" />
     <parent
@@ -674,5 +666,5 @@
       link="trailer" />
     <axis
-      xyz="0 0 1" />
+      xyz="0 1 0" />
   </joint>
   <link
@@ -680,15 +672,15 @@
     <inertial>
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
Commit message: trying to resolve issue with joint transformations

File: urdf/project_1_group_2.urdf.xacro (robot description, xacro)
@@ -35,4 +35,6 @@
       </visual>
   </xacro:macro>
+  # Add this before base link
+  <link name="dummy_link"></link>
   <link
     name="base_link">
@@ -75,4 +77,16 @@
     </collision>
   </link>
+    # Add this after base link
+  <joint
+    name="dummy_joint"
+    type="fixed">
+    <origin
+      rpy="0 0 0"
+      xyz="0 0 0" />
+    <parent
+      link="dummy_link"/>
+    <child
+      link="base_link"/>
+  </joint>
   <link
     name="steering_wheel_1">
@@ -201,5 +215,5 @@
         iyz="5.01717636400841E-07"
         izz="0.00664244711710664" />
-    </inertial>
+      </inertial>
     <visual>
       <origin
@@ -622,5 +636,5 @@
         rpy="0 0 0" />
       <mass
-        value=".5" />
+        value="0.5" />
       <inertia
         ixx="0.106926412723749"
@@ -826,57 +840,4 @@
     <axis
       xyz="0 0 0" />
-  </joint>
-  <link
-    name="lidar_link">
-    <inertial>
-      <origin
-        xyz="0 0.00127000000000005 0"
-        rpy="0 0 0" />
-      <mass
-        value="0.00514814798763055" />
-      <inertia
-        ixx="8.33112604888014E-07"
-        ixy="-3.20922964057601E-40"
-        ixz="0"
-        iyy="1.66068957784986E-06"
-        iyz="2.8186396765545E-40"
-        izz="8.33112604888014E-07" />
-    </inertial>
-    <visual>
-      <origin
-        xyz="0 0 0"
-        rpy="0 0 0" />
-      <geometry>
-        <mesh
-          filename="package://project_1_group_2/meshes/lidar_link.STL" />
-      </geometry>
-      <material
-        name="">
-        <color
-          rgba="0.792156862745098 0.819607843137255 0.933333333333333 1" />
-      </material>
-    </visual>
-    <collision>
-      <origin
-        xyz="0 0 0"
-        rpy="0 0 0" />
-      <geometry>
-        <mesh
-          filename="package://project_1_group_2/meshes/lidar_link.STL" />
-      </geometry>
-    </collision>
-  </link>
-  <joint
-    name="lidar_joint"
-    type="continuous">
-    <origin
-      xyz="0.219541699413715 -0.521188368096002 0.439623181973066"
-      rpy="1.5707963267949 0 0" />
-    <parent
-      link="base_link" />
-    <child
-      link="lidar_link" />
-    <axis
-      xyz="0 1 0" />
   </joint>
   <ros2_control name="GazeboSystem" type="system">

Commit message: added competition track and files

File: urdf/project_1_group_2.urdf.xacro (robot description, xacro)
@@ -840,4 +840,57 @@
     <axis
       xyz="0 0 0" />
+  </joint>
+    <link
+    name="lidar_link">
+    <inertial>
+      <origin
+        xyz="0 0.00127000000000005 0"
+        rpy="0 0 0" />
+      <mass
+        value="0.00514814798763055" />
+      <inertia
+        ixx="8.33112604888014E-07"
+        ixy="-3.20922964057601E-40"
+        ixz="0"
+        iyy="1.66068957784986E-06"
+        iyz="2.8186396765545E-40"
+        izz="8.33112604888014E-07" />
+    </inertial>
+    <visual>
+      <origin
+        xyz="0 0 0"
+        rpy="0 0 0" />
+      <geometry>
+        <mesh
+          filename="package://project_1_group_2/meshes/lidar_link.STL" />
+      </geometry>
+      <material
+        name="">
+        <color
+          rgba="0.792156862745098 0.819607843137255 0.933333333333333 1" />
+      </material>
+    </visual>
+    <collision>
+      <origin
+        xyz="0 0 0"
+        rpy="0 0 0" />
+      <geometry>
+        <mesh
+          filename="package://project_1_group_2/meshes/lidar_link.STL" />
+      </geometry>
+    </collision>
+  </link>
+  <joint
+    name="lidar_joint"
+    type="continuous">
+    <origin
+      xyz="0.219541699413715 -0.521188368096002 0.439623181973066"
+      rpy="1.5707963267949 0 0" />
+    <parent
+      link="base_link" />
+    <child
+      link="lidar_link" />
+    <axis
+      xyz="0 1 0" />
   </joint>
   <ros2_control name="GazeboSystem" type="system">

Commit message: proportional controller working to reach points (10,10)

File: urdf/project_1_group_2.urdf.xacro (robot description, xacro)
@@ -96,5 +96,5 @@
         rpy="0 0 0" />
       <mass
-        value="5.295424107267105" />
+        value="15.295424107267105" />
       <inertia
         ixx="0.000710809060839366"
@@ -154,5 +154,5 @@
         rpy="0 0 0" />
       <mass
-        value="0.217134053712094" />
+        value="2.217134053712094" />
       <inertia
         ixx="0.000126052696684198"
@@ -260,5 +260,5 @@
         rpy="0 0 0" />
       <mass
-        value="5.295424107267105" />
+        value="15.295424107267105" />
       <inertia
         ixx="0.000710809060839365"
@@ -318,5 +318,5 @@
         rpy="0 0 0" />
       <mass
-        value="0.217134053712094" />
+        value="2.217134053712094" />
       <inertia
         ixx="0.000126052696684198"
@@ -841,5 +841,5 @@
       xyz="0 0 0" />
   </joint>
-    <link
+  <link
     name="lidar_link">
     <inertial>
